File: bt-trx-dev-board.kicad_pcb (KiCad board)
At the start: 2 copper layers, 78 x 68 mm, 59 parts, among them J1 RJ45, J10 Conn_01x08, J2 PTT_BUTTON, J3 PTT_CON, J4 Conn_01x02, J5 PTT_SEL, J6 I2C, J7 Conn_01x02, J8 I2C, J9 Conn_01x08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

Commit message: Add VIAs on test points for better alignment [#21]
Routing:
- net GNDA: vias 0 -> 1
- net GND: vias 0 -> 1
- net /A_OUT_LP: vias 0 -> 1
- net /A_OUT_LN: vias 0 -> 1
- net /A_IN_LP: vias 0 -> 1
- net /A_IN_LN: vias 0 -> 1
- net /AUDIO_OUT_MIC: vias 0 -> 1
- net /AUDIO_IN_SPK: vias 0 -> 1
Changed lines of the file:
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@@
     (thickness 1.6)
     (drawings 881)
-    (tracks 361)
+    (tracks 377)
     (zones 0)
     (modules 59)
@@
   (gr_line (start 198.425 129.3) (end 198.425 69.342) (layer Edge.Cuts) (width 0.2))
   (gr_line (start 120.425 66.3) (end 120.42331 132.325) (layer Edge.Cuts) (width 0.2))
+  (via (at 152.908 67.818) (size 0.8) (drill 0.4) (layers F.Cu B.Cu) (net 1))
   (via (at 151.892 131.826) (size 0.8) (drill 0.4) (layers F.Cu B.Cu) (net 30))
   (via (at 140.97 131.826) (size 0.8) (drill 0.4) (layers F.Cu B.Cu) (net 30))
@@
   (segment (start 124.4055 85.9245) (end 124.46 85.979) (width 0.25) (layer F.Cu) (net 25))
   (segment (start 124.4055 83.566) (end 124.4055 85.9245) (width 0.25) (layer F.Cu) (net 25))
+  (segment (start 124.46 85.979) (end 124.46 85.979) (width 0.25) (layer F.Cu) (net 25))
+  (via (at 124.46 85.979) (size 0.8) (drill 0.4) (layers F.Cu B.Cu) (net 25))
   (segment (start 135.89 82.395) (end 135.89 80.645) (width 0.25) (layer F.Cu) (net 26))
   (segment (start 134.719 83.566) (end 135.89 82.395) (width 0.25) (layer F.Cu) (net 26))
@@
   (segment (start 129.9845 85.9155) (end 130.048 85.979) (width 0.25) (layer F.Cu) (net 27))
   (segment (start 129.9845 83.566) (end 129.9845 85.9155) (width 0.25) (layer F.Cu) (net 27))
+  (segment (start 130.048 85.979) (end 130.048 85.979) (width 0.25) (layer F.Cu) (net 27))
+  (via (at 130.048 85.979) (size 0.8) (drill 0.4) (layers F.Cu B.Cu) (net 27))
   (segment (start 161.29 78.17) (end 161.29 81.28) (width 0.25) (layer F.Cu) (net 28))
   (segment (start 161.29 77.47) (end 161.29 78.17) (width 0.25) (layer F.Cu) (net 28))
@@
   (segment (start 163.3855 81.2345) (end 163.34 81.28) (width 0.25) (layer F.Cu) (net 29))
   (segment (start 163.3855 78.74) (end 163.3855 81.2345) (width 0.25) (layer F.Cu) (net 29))
+  (segment (start 163.3855 78.74) (end 163.3855 78.74) (width 0.25) (layer F.Cu) (net 29))
+  (via (at 163.3855 78.74) (size 0.8) (drill 0.4) (layers F.Cu B.Cu) (net 29))
   (segment (start 134.569 88.0655) (end 134.569 89.5655) (width 0.5) (layer F.Cu) (net 30))
   (segment (start 136.239966 87.63) (end 135.0045 87.63) (width 0.5) (layer F.Cu) (net 30))
@@
   (segment (start 163.3855 76.2) (end 162.814 76.2) (width 0.25) (layer F.Cu) (net 34))
   (segment (start 162.814 76.2) (end 162.56 75.946) (width 0.25) (layer F.Cu) (net 34))
+  (segment (start 163.3855 76.2) (end 163.3855 76.2) (width 0.25) (layer F.Cu) (net 34))
+  (via (at 163.3855 76.2) (size 0.8) (drill 0.4) (layers F.Cu B.Cu) (net 34))
   (segment (start 182.372 86.36) (end 179.07 86.36) (width 0.5) (layer F.Cu) (net 35))
   (segment (start 189.23 83.82) (end 184.912 83.82) (width 0.5) (layer F.Cu) (net 35))
@@
   (segment (start 162.1155 72.39) (end 163.3855 73.66) (width 0.25) (layer F.Cu) (net 47))
   (segment (start 161.29 72.39) (end 162.1155 72.39) (width 0.25) (layer F.Cu) (net 47))
+  (segment (start 163.3855 73.66) (end 163.3855 73.66) (width 0.25) (layer F.Cu) (net 47))
+  (segment (start 163.3855 73.66) (end 163.3855 73.66) (width 0.25) (layer F.Cu) (net 47))
+  (via (at 163.3855 73.66) (size 0.8) (drill 0.4) (layers F.Cu B.Cu) (net 47))
   (segment (start 175.514 75.45) (end 174.486 74.422) (width 0.25) (layer F.Cu) (net 48))
   (segment (start 175.514 77.2) (end 175.514 75.45) (width 0.25) (layer F.Cu) (net 48))
@@
   (segment (start 127 85.725) (end 127.254 85.979) (width 0.25) (layer F.Cu) (net 50))
   (segment (start 127 80.645) (end 127 85.725) (width 0.25) (layer F.Cu) (net 50))
+  (segment (start 127.254 85.979) (end 127.254 85.979) (width 0.25) (layer F.Cu) (net 50))
+  (via (at 127.254 85.979) (size 0.8) (drill 0.4) (layers F.Cu B.Cu) (net 50))
   (segment (start 129.569 88.19134) (end 129.569 89.5655) (width 0.25) (layer F.Cu) (net 51))
   (segment (start 132.25166 87.63) (end 130.13034 87.63) (width 0.25) (layer F.Cu) (net 51))
@@
   (segment (start 134.747 84.074) (end 132.842 85.979) (width 0.25) (layer F.Cu) (net 51))
   (segment (start 139.291 84.074) (end 134.747 84.074) (width 0.25) (layer F.Cu) (net 51))
+  (segment (start 132.842 85.979) (end 132.842 85.979) (width 0.25) (layer F.Cu) (net 51))
+  (via (at 132.842 85.979) (size 0.8) (drill 0.4) (layers F.Cu B.Cu) (net 51))
   (zone (net 1) (net_name GND) (layer F.Cu) (hatch edge 0.508)
     (connect_pads (clearance 0.2))
