File: bt-trx-dev-board.kicad_sch (KiCad schematic)
At the start: 18 parts, among them J1 RJ45, J10 JMP_CON_TRX, J2 PTT_BUTTON, J3 PTT_CON, J5 PTT_SEL, J9 JMP_CON, U1 FMB100, U2 LTV-816S

Commit message: anm: Added FMB100 to PCB
* Replaced WT32i with FMB100
* Swapped RX and TX transformers
* Removed MIC Bias C
Parts:
- removed C4: (no value), symbol Device:C
- C8, C9: value (none) -> 100nF; footprint (none) -> Capacitor_SMD:C_0805_2012Metric_Pad1.15x1.40mm_HandSolder
- R1: value (none) -> 10k; footprint (none) -> Resistor_SMD:R_0805_2012Metric_Pad1.15x1.40mm_HandSolder
- R8: value (none) -> 220R; footprint (none) -> Resistor_SMD:R_0805_2012Metric_Pad1.15x1.40mm_HandSolder
- U1: footprint (none) -> FMB100:FMB100
Connections:
- net +3.3V is gone; now on net +3V3: U1.2 (VBAT), U1.5 (VCC_IO)
- no-connect marks 16 -> 17
Other:
- note added: "PullUp RST permanently or connect it to uC?"
Changed lines of the file:
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@@
   (no_connect (at 74.93 49.53))
   (no_connect (at 74.93 62.23))
+  (no_connect (at 116.84 54.61))
   (no_connect (at 116.84 46.99))
   (no_connect (at 116.84 44.45))
@@
     (stroke (width 0) (type default) (color 0 0 0 0))
   )
-  (wire (pts (xy 116.84 54.61) (xy 130.81 54.61))
-    (stroke (width 0) (type default) (color 0 0 0 0))
-  )
   (wire (pts (xy 224.79 138.43) (xy 224.79 143.51))
-    (stroke (width 0) (type default) (color 0 0 0 0))
-  )
-  (wire (pts (xy 140.97 54.61) (xy 140.97 55.88))
-    (stroke (width 0) (type default) (color 0 0 0 0))
-  )
-  (wire (pts (xy 138.43 54.61) (xy 140.97 54.61))
     (stroke (width 0) (type default) (color 0 0 0 0))
   )
@@
   )
   (text "Connection to Transceiver" (at 17.78 121.92 0)
+    (effects (font (size 1.27 1.27)) (justify left bottom))
+  )
+  (text "PullUp RST permanently or connect it to uC?" (at 102.87 72.39 0)
     (effects (font (size 1.27 1.27)) (justify left bottom))
   )
@@
       (effects (font (size 1.27 1.27)) hide)
     )
-    (property "Value" "" (id 1) (at 191.77 109.22 90))
+    (property "Value" "+3V3" (id 1) (at 191.77 109.22 90))
     (property "Footprint" "" (id 2) (at 191.77 114.3 0)
       (effects (font (size 1.27 1.27)) hide)
@@
       (effects (font (size 1.27 1.27)) (justify left))
     )
-    (property "Value" "" (id 1) (at 189.992 119.507 0)
-      (effects (font (size 1.27 1.27)) (justify left))
-    )
-    (property "Footprint" "" (id 2) (at 193.548 120.65 90)
+    (property "Value" "10k" (id 1) (at 189.992 119.507 0)
+      (effects (font (size 1.27 1.27)) (justify left))
+    )
+    (property "Footprint" "Resistor_SMD:R_0805_2012Metric_Pad1.15x1.40mm_HandSolder" (id 2) (at 193.548 120.65 90)
       (effects (font (size 1.27 1.27)) hide)
     )
@@
       (effects (font (size 1.27 1.27)) (justify left))
     )
-    (property "Value" "" (id 1) (at 232.918 135.763 0)
-      (effects (font (size 1.27 1.27)) (justify left))
-    )
-    (property "Footprint" "" (id 2) (at 229.362 134.62 90)
+    (property "Value" "220R" (id 1) (at 232.918 135.763 0)
+      (effects (font (size 1.27 1.27)) (justify left))
+    )
+    (property "Footprint" "Resistor_SMD:R_0805_2012Metric_Pad1.15x1.40mm_HandSolder" (id 2) (at 229.362 134.62 90)
       (effects (font (size 1.27 1.27)) hide)
     )
@@
     )
     (property "Datasheet" "" (id 3) (at 123.19 41.91 0)
-      (effects (font (size 1.27 1.27)) hide)
-    )
-    (pin "1")
-  )
-  (symbol (lib_id "power:GNDPWR") (at 140.97 55.88 0) (unit 1)
-    (in_bom yes) (on_board yes)
-    (property "Reference" "#PWR014" (id 0) (at 140.97 60.96 0)
-      (effects (font (size 1.27 1.27)) hide)
-    )
-    (property "Value" "GNDPWR" (id 1) (at 141.0716 59.7916 0))
-    (property "Footprint" "" (id 2) (at 140.97 57.15 0)
-      (effects (font (size 1.27 1.27)) hide)
-    )
-    (property "Datasheet" "" (id 3) (at 140.97 57.15 0)
       (effects (font (size 1.27 1.27)) hide)
     )
@@
   (symbol (lib_id "Device:C") (at 44.45 93.98 180) (unit 1)
     (in_bom yes) (on_board yes)
-    (property "Reference" "C?" (id 0) (at 50.8508 93.98 90))
-    (property "Value" "" (id 1) (at 48.5394 93.98 90))
-    (property "Footprint" "" (id 2) (at 43.4848 90.17 0)
+    (property "Reference" "C9" (id 0) (at 50.8508 93.98 90))
+    (property "Value" "100nF" (id 1) (at 48.5394 93.98 90))
+    (property "Footprint" "Capacitor_SMD:C_0805_2012Metric_Pad1.15x1.40mm_HandSolder" (id 2) (at 43.4848 90.17 0)
       (effects (font (size 1.27 1.27)) hide)
     )
@@
   (symbol (lib_id "Device:C") (at 33.02 93.98 180) (unit 1)
     (in_bom yes) (on_board yes)
-    (property "Reference" "C?" (id 0) (at 39.4208 93.98 90))
-    (property "Value" "" (id 1) (at 37.1094 93.98 90))
-    (property "Footprint" "" (id 2) (at 32.0548 90.17 0)
+    (property "Reference" "C8" (id 0) (at 39.4208 93.98 90))
+    (property "Value" "100nF" (id 1) (at 37.1094 93.98 90))
+    (property "Footprint" "Capacitor_SMD:C_0805_2012Metric_Pad1.15x1.40mm_HandSolder" (id 2) (at 32.0548 90.17 0)
       (effects (font (size 1.27 1.27)) hide)
     )
@@
     )
     (pin "1")
-  )
-  (symbol (lib_id "Device:C") (at 134.62 54.61 270) (unit 1)
-    (in_bom yes) (on_board yes)
-    (property "Reference" "C?" (id 0) (at 134.62 48.2092 90))
-    (property "Value" "" (id 1) (at 134.62 50.5206 90))
-    (property "Footprint" "" (id 2) (at 130.81 55.5752 0)
-      (effects (font (size 1.27 1.27)) hide)
-    )
-    (property "Datasheet" "~" (id 3) (at 134.62 54.61 0)
-      (effects (font (size 1.27 1.27)) hide)
-    )
-    (property "Mouser Best.Nr." "80-C0805C105K3RAUTO" (id 4) (at -39.37 10.16 0)
-      (effects (font (size 1.27 1.27)) hide)
-    )
-    (property "PartNrDigikey" "399-6929-1-ND" (id 5) (at 134.62 54.61 0)
-      (effects (font (size 1.27 1.27)) hide)
-    )
-    (pin "1")
-    (pin "2")
   )
   (symbol (lib_id "power:GND") (at 31.75 133.35 0) (unit 1)
@@
     (pin "8")
   )
-  (symbol (lib_id "power:+3.3V") (at 68.58 39.37 90) (unit 1)
-    (in_bom yes) (on_board yes)
-    (property "Reference" "#PWR?" (id 0) (at 72.39 39.37 0)
-      (effects (font (size 1.27 1.27)) hide)
-    )
-    (property "Value" "+3.3V" (id 1) (at 64.77 39.37 90)
-      (effects (font (size 1.27 1.27)) (justify left))
-    )
-    (property "Footprint" "" (id 2) (at 68.58 39.37 0)
-      (effects (font (size 1.27 1.27)) hide)
-    )
-    (property "Datasheet" "" (id 3) (at 68.58 39.37 0)
-      (effects (font (size 1.27 1.27)) hide)
-    )
-    (pin "1")
-  )
   (symbol (lib_id "fbm100:FMB100") (at 96.52 50.8 0) (unit 1)
     (in_bom yes) (on_board yes) (fields_autoplaced)
     (property "Reference" "U1" (id 0) (at 95.885 30.7172 0))
     (property "Value" "FMB100" (id 1) (at 95.885 33.2541 0))
-    (property "Footprint" "" (id 2) (at 80.01 30.48 0)
+    (property "Footprint" "FMB100:FMB100" (id 2) (at 80.01 30.48 0)
       (effects (font (size 1.27 1.27)) hide)
     )
@@
     (pin "9")
   )
+  (symbol (lib_id "power:+3V3") (at 68.58 39.37 90) (unit 1)
+    (in_bom yes) (on_board yes)
+    (property "Reference" "#PWR0103" (id 0) (at 72.39 39.37 0)
+      (effects (font (size 1.27 1.27)) hide)
+    )
+    (property "Value" "+3V3" (id 1) (at 62.23 39.37 90))
+    (property "Footprint" "" (id 2) (at 68.58 39.37 0)
+      (effects (font (size 1.27 1.27)) hide)
+    )
+    (property "Datasheet" "" (id 3) (at 68.58 39.37 0)
+      (effects (font (size 1.27 1.27)) hide)
+    )
+    (pin "1")
+  )
+  (symbol (lib_id "power:+3V3") (at 68.58 46.99 90) (unit 1)
+    (in_bom yes) (on_board yes)
+    (property "Reference" "#PWR0105" (id 0) (at 72.39 46.99 0)
+      (effects (font (size 1.27 1.27)) hide)
+    )
+    (property "Value" "+3V3" (id 1) (at 62.23 46.99 90))
+    (property "Footprint" "" (id 2) (at 68.58 46.99 0)
+      (effects (font (size 1.27 1.27)) hide)
+    )
+    (property "Datasheet" "" (id 3) (at 68.58 46.99 0)
+      (effects (font (size 1.27 1.27)) hide)
+    )
+    (pin "1")
+  )
   (symbol (lib_id "power:GNDPWR") (at 69.85 52.07 270) (unit 1)
     (in_bom yes) (on_board yes)
-    (property "Reference" "#PWR?" (id 0) (at 64.77 52.07 0)
+    (property "Reference" "#PWR0104" (id 0) (at 64.77 52.07 0)
       (effects (font (size 1.27 1.27)) hide)
     )
@@
     )
     (property "Datasheet" "" (id 3) (at 68.58 52.07 0)
-      (effects (font (size 1.27 1.27)) hide)
-    )
-    (pin "1")
-  )
-  (symbol (lib_id "power:+3.3V") (at 68.58 46.99 90) (unit 1)
-    (in_bom yes) (on_board yes)
-    (property "Reference" "#PWR?" (id 0) (at 72.39 46.99 0)
-      (effects (font (size 1.27 1.27)) hide)
-    )
-    (property "Value" "+3.3V" (id 1) (at 64.77 46.99 90)
-      (effects (font (size 1.27 1.27)) (justify left))
-    )
-    (property "Footprint" "" (id 2) (at 68.58 46.99 0)
-      (effects (font (size 1.27 1.27)) hide)
-    )
-    (property "Datasheet" "" (id 3) (at 68.58 46.99 0)
       (effects (font (size 1.27 1.27)) hide)
     )
@@
       (reference "#PWR013") (unit 1) (value "+3V3") (footprint "")
     )
-    (path "/00000000-0000-0000-0000-00005e253cb8"
-      (reference "#PWR014") (unit 1) (value "GNDPWR") (footprint "")
-    )
     (path "/00000000-0000-0000-0000-00005e2639f5"
       (reference "#PWR015") (unit 1) (value "GNDPWR") (footprint "")
@@
       (reference "#PWR0102") (unit 1) (value "+3V3") (footprint "")
     )
-    (path "/06476481-e551-479d-8dcd-8e30ad86ebea"
-      (reference "#PWR?") (unit 1) (value "+3.3V") (footprint "")
+    (path "/4ce942e7-985c-447f-ab38-83ccfc33c647"
+      (reference "#PWR0103") (unit 1) (value "+3V3") (footprint "")
     )
     (path "/c85a46e9-9b74-4ad4-954e-bc404659f9f8"
-      (reference "#PWR?") (unit 1) (value "GNDPWR") (footprint "")
-    )
-    (path "/ceaf894b-9462-4693-ba67-7ec81a591449"
-      (reference "#PWR?") (unit 1) (value "+3.3V") (footprint "")
+      (reference "#PWR0104") (unit 1) (value "GNDPWR") (footprint "")
+    )
+    (path "/9c46b331-b58e-4049-8d56-737f06837c43"
+      (reference "#PWR0105") (unit 1) (value "+3V3") (footprint "")
     )
     (path "/00000000-0000-0000-0000-00005be3535b/00000000-0000-0000-0000-00005e2ad650"
       (reference "C3") (unit 1) (value "1uF") (footprint "Capacitor_SMD:C_0805_2012Metric_Pad1.15x1.40mm_HandSolder")
     )
-    (path "/00000000-0000-0000-0000-00005e304ad9"
-      (reference "C4") (unit 1) (value "1uF") (footprint "Capacitor_SMD:C_0805_2012Metric_Pad1.15x1.40mm_HandSolder")
-    )
     (path "/00000000-0000-0000-0000-00005be3535b/00000000-0000-0000-0000-00005bfc0ac9"
       (reference "C5") (unit 1) (value "15pF") (footprint "Capacitor_SMD:C_0805_2012Metric_Pad1.15x1.40mm_HandSolder")
@@
     )
     (path "/30519ad1-4770-4e8d-a0b9-f77f1abb5e9a"
-      (reference "U1") (unit 1) (value "FMB100") (footprint "")
+      (reference "U1") (unit 1) (value "FMB100") (footprint "FMB100:FMB100")
     )
     (path "/00000000-0000-0000-0000-00005e115f72"
