File: bt-trx-dev-board.kicad_sch (KiCad schematic)
At the start: 17 parts, among them J1 RJ45, J10 JMP_CON_TRX, J2 PTT_BUTTON, J3 PTT_CON, J5 PTT_SEL, J9 JMP_CON, U1 FMB100, U2 LTV-816S

Commit message: am: Modified HW indication voltage
* Added R10 for voltage divider (v6.x == 1.65V)
* Replaced all R footprints with current ones from KiCad lib
Parts:
- R1, R8: footprint Resistor_SMD:R_0805_2012Metric_Pad1.15x1.40mm_HandSolder -> Resistor_SMD:R_0805_2012Metric_Pad1.20x1.40mm_HandSolder
Changed lines of the file:
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@@
       (effects (font (size 1.27 1.27)) (justify left))
     )
-    (property "Footprint" "Resistor_SMD:R_0805_2012Metric_Pad1.15x1.40mm_HandSolder" (id 2) (at 193.548 120.65 90)
+    (property "Footprint" "Resistor_SMD:R_0805_2012Metric_Pad1.20x1.40mm_HandSolder" (id 2) (at 193.548 120.65 90)
       (effects (font (size 1.27 1.27)) hide)
     )
@@
       (effects (font (size 1.27 1.27)) (justify left))
     )
-    (property "Footprint" "Resistor_SMD:R_0805_2012Metric_Pad1.15x1.40mm_HandSolder" (id 2) (at 229.362 134.62 90)
+    (property "Footprint" "Resistor_SMD:R_0805_2012Metric_Pad1.20x1.40mm_HandSolder" (id 2) (at 229.362 134.62 90)
       (effects (font (size 1.27 1.27)) hide)
     )
@@
       (reference "#PWR02") (unit 1) (value "GND") (footprint "")
     )
+    (path "/00000000-0000-0000-0000-00005c10b93a/5a6d95b3-6591-4e58-9826-13bf242ab2db"
+      (reference "#PWR03") (unit 1) (value "GNDPWR") (footprint "")
+    )
     (path "/00000000-0000-0000-0000-00005e273431"
       (reference "#PWR04") (unit 1) (value "GNDPWR") (footprint "")
@@
     )
     (path "/00000000-0000-0000-0000-00005cd1bcf6"
-      (reference "R1") (unit 1) (value "10k") (footprint "Resistor_SMD:R_0805_2012Metric_Pad1.15x1.40mm_HandSolder")
+      (reference "R1") (unit 1) (value "10k") (footprint "Resistor_SMD:R_0805_2012Metric_Pad1.20x1.40mm_HandSolder")
     )
     (path "/00000000-0000-0000-0000-00005c10b93a/00000000-0000-0000-0000-00005d9f2fe4"
-      (reference "R2") (unit 1) (value "10k") (footprint "Resistor_SMD:R_0805_2012Metric_Pad1.15x1.40mm_HandSolder")
+      (reference "R2") (unit 1) (value "10k") (footprint "Resistor_SMD:R_0805_2012Metric_Pad1.20x1.40mm_HandSolder")
     )
     (path "/00000000-0000-0000-0000-00005c10b93a/00000000-0000-0000-0000-00005c012726"
-      (reference "R3") (unit 1) (value "2.2k") (footprint "Resistor_SMD:R_0805_2012Metric_Pad1.15x1.40mm_HandSolder")
+      (reference "R3") (unit 1) (value "2.2k") (footprint "Resistor_SMD:R_0805_2012Metric_Pad1.20x1.40mm_HandSolder")
     )
     (path "/00000000-0000-0000-0000-00005c10b93a/00000000-0000-0000-0000-00005c1540d9"
-      (reference "R4") (unit 1) (value "820R") (footprint "Resistor_SMD:R_0805_2012Metric_Pad1.15x1.40mm_HandSolder")
+      (reference "R4") (unit 1) (value "820R") (footprint "Resistor_SMD:R_0805_2012Metric_Pad1.20x1.40mm_HandSolder")
     )
     (path "/00000000-0000-0000-0000-00005c10b93a/00000000-0000-0000-0000-00005c1540f1"
-      (reference "R5") (unit 1) (value "820R") (footprint "Resistor_SMD:R_0805_2012Metric_Pad1.15x1.40mm_HandSolder")
+      (reference "R5") (unit 1) (value "820R") (footprint "Resistor_SMD:R_0805_2012Metric_Pad1.20x1.40mm_HandSolder")
     )
     (path "/00000000-0000-0000-0000-00005c10b93a/00000000-0000-0000-0000-00005c81c8a6"
-      (reference "R6") (unit 1) (value "4.7k") (footprint "Resistor_SMD:R_0805_2012Metric_Pad1.15x1.40mm_HandSolder")
+      (reference "R6") (unit 1) (value "4.7k") (footprint "Resistor_SMD:R_0805_2012Metric_Pad1.20x1.40mm_HandSolder")
     )
     (path "/00000000-0000-0000-0000-00005c10b93a/00000000-0000-0000-0000-00005c81c972"
-      (reference "R7") (unit 1) (value "4.7k") (footprint "Resistor_SMD:R_0805_2012Metric_Pad1.15x1.40mm_HandSolder")
+      (reference "R7") (unit 1) (value "4.7k") (footprint "Resistor_SMD:R_0805_2012Metric_Pad1.20x1.40mm_HandSolder")
     )
     (path "/00000000-0000-0000-0000-00005e1205ef"
-      (reference "R8") (unit 1) (value "220R") (footprint "Resistor_SMD:R_0805_2012Metric_Pad1.15x1.40mm_HandSolder")
+      (reference "R8") (unit 1) (value "220R") (footprint "Resistor_SMD:R_0805_2012Metric_Pad1.20x1.40mm_HandSolder")
     )
     (path "/00000000-0000-0000-0000-00005c10b93a/00000000-0000-0000-0000-00005e288a63"
-      (reference "R9") (unit 1) (value "10k") (footprint "Resistor_SMD:R_0805_2012Metric_Pad1.15x1.40mm_HandSolder")
+      (reference "R9") (unit 1) (value "10k") (footprint "Resistor_SMD:R_0805_2012Metric_Pad1.20x1.40mm_HandSolder")
+    )
+    (path "/00000000-0000-0000-0000-00005c10b93a/2cd62f0c-c86a-46e3-b421-c11b52f903e6"
+      (reference "R10") (unit 1) (value "10k") (footprint "Resistor_SMD:R_0805_2012Metric_Pad1.20x1.40mm_HandSolder")
     )
     (path "/00000000-0000-0000-0000-00005be3535b/00000000-0000-0000-0000-00005c774d1e"

Commit message: am: Connected FMB100 RST pin to ESP
* Connected FMB100 RST pin to ESP in schematic and PCB
Connections:
- net FMB_RST_FROM_UC: now reaches U1.19 (PIO1/RSTN)
- net WT32_ONOFF_FROM_UC renamed FMB_ONOFF_FROM_UC
- no-connect marks 17 -> 16
Other:
- sheet Microcontroller ports: added FMB_ONOFF_FROM_UC, FMB_RST_FROM_UC; removed WT32_ONOFF_FROM_UC
- note removed: "Add LED to PIO60 acc. ref. design?"
- note removed: "PullUp RST permanently or connect it to uC?"
Changed lines of the file:
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@@
   (no_connect (at 74.93 64.77))
   (no_connect (at 100.33 69.85))
-  (no_connect (at 102.87 69.85))
   (no_connect (at 74.93 54.61))
   (no_connect (at 97.79 69.85))
@@
     (stroke (width 0) (type default) (color 0 0 0 0))
   )
+  (wire (pts (xy 212.09 92.71) (xy 214.63 92.71))
+    (stroke (width 0) (type default) (color 0 0 0 0))
+  )
   (wire (pts (xy 33.02 87.63) (xy 33.02 90.17))
     (stroke (width 0) (type default) (color 0 0 0 0))
@@
   )
   (wire (pts (xy 214.63 83.82) (xy 212.09 83.82))
+    (stroke (width 0) (type default) (color 0 0 0 0))
+  )
+  (wire (pts (xy 102.87 69.85) (xy 102.87 76.2))
     (stroke (width 0) (type default) (color 0 0 0 0))
   )
@@
     (effects (font (size 1.27 1.27)) (justify left bottom))
   )
-  (text "PullUp RST permanently or connect it to uC?" (at 102.87 72.39 0)
-    (effects (font (size 1.27 1.27)) (justify left bottom))
-  )
-  (text "Add LED to PIO60 acc. ref. design?" (at 38.1 59.69 0)
-    (effects (font (size 1.27 1.27)) (justify left bottom))
-  )
   (label "UC_PTT_LED" (at 191.77 133.35 0)
     (effects (font (size 1.27 1.27)) (justify left bottom))
@@
     (effects (font (size 1.27 1.27)) (justify right bottom))
   )
+  (label "FMB_RST_FROM_UC" (at 212.09 92.71 180)
+    (effects (font (size 1.27 1.27)) (justify right bottom))
+  )
   (label "A_IN_LP" (at 121.92 49.53 0)
     (effects (font (size 1.27 1.27)) (justify left bottom))
@@
     (effects (font (size 1.27 1.27)) (justify right bottom))
   )
-  (label "WT32_ONOFF_FROM_UC" (at 212.09 90.17 180)
+  (label "FMB_ONOFF_FROM_UC" (at 212.09 90.17 180)
     (effects (font (size 1.27 1.27)) (justify right bottom))
   )
@@
     (effects (font (size 1.27 1.27)) (justify left bottom))
   )
-  (label "WT32_ONOFF_FROM_UC" (at 69.85 41.91 180)
+  (label "FMB_ONOFF_FROM_UC" (at 69.85 41.91 180)
     (effects (font (size 1.27 1.27)) (justify right bottom))
   )
@@
   (label "A_OUT_LP" (at 121.92 57.15 0)
     (effects (font (size 1.27 1.27)) (justify left bottom))
+  )
+  (label "FMB_RST_FROM_UC" (at 102.87 76.2 270)
+    (effects (font (size 1.27 1.27)) (justify right bottom))
   )
   (label "UC_PTT_LED" (at 212.09 86.36 180)
@@
       (effects (font (size 1.27 1.27)) (justify left))
     )
-    (pin "WT32_ONOFF_FROM_UC" output (at 214.63 90.17 180)
-      (effects (font (size 1.27 1.27)) (justify left))
-    )
     (pin "+V_IN" input (at 214.63 66.04 180)
       (effects (font (size 1.27 1.27)) (justify left))
@@
       (effects (font (size 1.27 1.27)) (justify right))
     )
-  )
+    (pin "FMB_ONOFF_FROM_UC" output (at 214.63 90.17 180)
+      (effects (font (size 1.27 1.27)) (justify left))
+    )
+    (pin "FMB_RST_FROM_UC" output (at 214.63 92.71 180)
+      (effects (font (size 1.27 1.27)) (justify left))
+    )
+  )
